Commit message: Modified URDF to match NW's setup. Joint limits were bad.

File: mico-modified-working.urdf (robot description, URDF)
Before this commit: robot ADA, 17 links, 16 joints
Joints:
- joint mico_joint_1: limit lower=-3.6652 upper=0.52360 effort=18 velocity=0.94 -> lower=-0.52360 upper=3.6652 effort=18 velocity=0.94
- joint mico_joint_2: limit lower=2.46 upper=5.26 effort=18 velocity=0.94 -> lower=-2.1 upper=0.7 effort=18 velocity=0.94
- joint mico_joint_3: limit lower=0.65 upper=4.01 effort=18 velocity=0.94 -> lower=-0.86841 upper=2.4916 effort=18 velocity=0.94
